File: board/telescope_dew_heater/telescope_dew_heater.kicad_sch (KiCad schematic)
At the start: 9 parts, among them J1 RCA1, Q1 Q_NMOS_GDS, U1 NE555P

Commit message: Updated some footprints
Parts:
- J1: footprint (none) -> Connector_PinHeader_2.54mm:PinHeader_1x02_P2.54mm_Vertical
- Q1: footprint (none) -> Package_TO_SOT_THT:TO-251-3_Vertical
- RV1: value R_Potentiometer_US -> POTENTIOMETER
Changed lines of the file:
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@@
       (effects (font (size 1.27 1.27)) (justify left))
     )
-    (property "Footprint" "" (at 204.47 33.02 0)
+    (property "Footprint" "Connector_PinHeader_2.54mm:PinHeader_1x02_P2.54mm_Vertical" (at 204.47 33.02 0)
       (effects (font (size 1.27 1.27)) hide)
     )
@@
       (effects (font (size 1.27 1.27)))
     )
-    (property "Value" "R_Potentiometer_US" (at 203.2 71.12 90)
+    (property "Value" "POTENTIOMETER" (at 201.93 71.12 90)
       (effects (font (size 1.27 1.27)))
     )
@@
       (effects (font (size 1.27 1.27)) (justify left))
     )
-    (property "Footprint" "" (at 207.01 43.18 0)
+    (property "Footprint" "Package_TO_SOT_THT:TO-251-3_Vertical" (at 207.01 43.18 0)
       (effects (font (size 1.27 1.27)) hide)
     )
