File: board/telescope_dew_heater/telescope_dew_heater.kicad_sch (KiCad schematic)
At the start: 38 parts, among them J1 RCA1, J2 RCA1, J3 RCA1, J4 RCA1, Q1 Q_NMOS_GDS, Q2 Q_NMOS_GDS, Q3 Q_NMOS_GDS, Q4 Q_NMOS_GDS, SW1 SW_DPDT_x2, U1 NE555P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

Commit message: Push update
Parts:
- removed C2, C5, C6: 0.1u, Capacitor_THT:C_Disc_D3.4mm_W2.1mm_P2.50mm, symbol Device:C
- removed C4, C7, C8: 68u, Capacitor_THT:CP_Radial_D6.3mm_P2.50mm, symbol Device:C_Polarized_US
- removed D2, D4, D5, D6, D7, D8: D, Diode_THT:D_DO-35_SOD27_P7.62mm_Horizontal, symbol Device:D
- removed J2, J3, J4: RCA1, Connector_PinHeader_2.54mm:PinHeader_1x02_P2.54mm_Vertical, symbol Connector:Conn_Coaxial
- removed Q2, Q3, Q4: Q_NMOS_GDS, Package_TO_SOT_THT:TO-251-3_Vertical, symbol Device:Q_NMOS_GDS
- removed R2, R3, R4: 1K, Resistor_THT:R_Axial_DIN0207_L6.3mm_D2.5mm_P7.62mm_Horizontal, symbol Device:R_US
- removed RV2, RV3, RV4: 100K POT, Connector_PinHeader_2.54mm:PinHeader_1x03_P2.54mm_Vertical, symbol Device:R_Potentiometer_US
- removed U2, U3, U4: NE555P, Package_DIP:DIP-8_W7.62mm, symbol Timer:NE555P
- renumbered D3 to D2
