File: board/telescope_dew_heater/_autosave-telescope_dew_heater.kicad_sch (KiCad schematic)
At the start: 38 parts, among them J1 RCA1, J2 RCA1, J3 RCA1, J4 RCA1, Q1 Q_NMOS_GDS, Q2 Q_NMOS_GDS, Q3 Q_NMOS_GDS, Q4 Q_NMOS_GDS, SW1 SW_DPDT_x2, U1 NE555P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

Commit message: Finished PWM controller schematic, started PCB layout
Todo: add power connector
Parts:
- renumbered C5 to C2, C7 to C4, C2 to C5, C4 to C7, D3 to D2, D5 to D3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
